File: lightPCB/lightPCB.kicad_pcb (KiCad board)
At the start: 2 copper layers, 59 x 30 mm, 24 parts, among them J1 I2C Connection, J2 Neopixel, U1 TCA6408APWR

Commit message: Replaced adafruit neopixel library with the fast led library to improve interrupt performace. Still having buzzes after timer runs out.
Other:
- board text added: "bkp515 QuizBoxFaceplate V1"
